File: robotics.sch (KiCad schematic (older format))
At the start: 3 parts, among them J1 RJ45, J2 Conn_01x03, J3 Conn_02x05_Odd_Even

Commit message: changed j1 to j3
Parts:
- removed J1: RJ45, symbol Connector:RJ45
- added J3: 8P8C, symbol Connector:8P8C
Changed lines of the file:
@@
 	4550 2150 4550 2950
 $Comp
-L Connector:RJ45 J1
-U 1 1 5C23E42B
+L Connector:8P8C J3
+U 1 1 5C5208BB
 P 1700 2300
-F 0 "J1" H 1755 2967 50  0000 C CNN
-F 1 "RJ45" H 1755 2876 50  0000 C CNN
+F 0 "J3" H 1755 2967 50  0000 C CNN
+F 1 "8P8C" H 1755 2876 50  0000 C CNN
 F 2 "" V 1700 2325 50  0001 C CNN
 F 3 "~" V 1700 2325 50  0001 C CNN
